File: MySensors MQ GasSensors Board/MQ_GasSensors_Board.brd (EAGLE design)
At the start: 16.5 x 38.1 mm, 5 parts

Commit message: Add hole to MQ sensors board; generate Gerbers
Routing:
- net A2: track 34.6 -> 37.8 mm
- net A3: track 27.0 -> 28.4 mm
Changed lines of the file:
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@@
 <?xml version="1.0" encoding="utf-8"?>
 <!DOCTYPE eagle SYSTEM "eagle.dtd">
-<eagle version="8.2.1">
+<eagle version="8.3.2">
 <drawing>
 <settings>
 <setting alwaysvectorfont="no"/>
+<setting keepoldvectorfont="yes"/>
 <setting verticaltext="up"/>
 </settings>
@@
 <text x="5.08" y="46.99" size="1.016" layer="22" font="vector" rot="MR270">MQ Sensor 2</text>
 <text x="5.08" y="27.305" size="1.016" layer="22" font="vector" rot="MR270">MQ Sensor 1</text>
-<text x="10.16" y="33.655" size="1.016" layer="21" font="vector" align="center">MQ Sensors Board
+<text x="10.16" y="34.925" size="1.016" layer="21" font="vector" align="center">MQ Sensors Board
 2017, R. Kainhofer</text>
+<hole x="10.16" y="31.75" drill="3.556"/>
 </plain>
 <attributes>
@@
 <wire x1="11.43" y1="12.7" x2="11.43" y2="13.97" width="0.1524" layer="1"/>
 <wire x1="11.43" y1="13.97" x2="10.16" y2="15.24" width="0.1524" layer="1"/>
-<wire x1="10.16" y1="15.24" x2="10.16" y2="43.18" width="0.1524" layer="1"/>
+<wire x1="10.16" y1="26.035" x2="10.16" y2="15.24" width="0.1524" layer="1"/>
+<wire x1="10.16" y1="43.18" x2="10.16" y2="37.465" width="0.1524" layer="1"/>
 <wire x1="10.16" y1="43.18" x2="7.62" y2="45.72" width="0.1524" layer="1"/>
+<wire x1="10.16" y1="37.465" x2="6.35" y2="33.655" width="0.1524" layer="1"/>
+<wire x1="6.35" y1="33.655" x2="6.35" y2="29.845" width="0.1524" layer="1"/>
+<wire x1="6.35" y1="29.845" x2="10.16" y2="26.035" width="0.1524" layer="1"/>
 </signal>
 <signal name="A3">
@@
 <contactref element="J1" pad="5"/>
 <wire x1="11.43" y1="15.24" x2="13.97" y2="12.7" width="0.1524" layer="1"/>
-<wire x1="11.43" y1="36.83" x2="11.43" y2="15.24" width="0.1524" layer="1"/>
-<wire x1="12.7" y1="38.1" x2="11.43" y2="36.83" width="0.1524" layer="1"/>
+<wire x1="11.43" y1="26.67" x2="11.43" y2="15.24" width="0.1524" layer="1"/>
+<wire x1="12.7" y1="38.1" x2="13.335" y2="38.1" width="0.1524" layer="1"/>
+<wire x1="13.335" y1="38.1" x2="13.97" y2="37.465" width="0.1524" layer="1"/>
+<wire x1="13.97" y1="37.465" x2="13.97" y2="29.21" width="0.1524" layer="1"/>
+<wire x1="13.97" y1="29.21" x2="11.43" y2="26.67" width="0.1524" layer="1"/>
 </signal>
 <signal name="A4">
